File: Design Files/40pin_AVRMCU.sch (KiCad schematic (older format))
At the start: 30 parts, among them CON1 USB-MINI-B, IC1 ATMEGA32-A, P1 CONN_5X2, P10 CONN_01X01, P2 CONN_10, P3 CONN_10, P4 CONN_10, P5 CONN_10, P6 CONN_01X01, P7 CONN_01X01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

Commit message: BOM updated
Parts:
- IC1: value ATMEGA32-A -> ATMEGA16
Changed lines of the file:
@@
 LIBS:contrib
 LIBS:valves
-LIBS:Starter_AVR-cache
 LIBS:40pin_AVRMCU-cache
 EELAYER 25 0
@@
 P 4175 3150
 F 0 "IC1" H 3325 5030 40  0000 L BNN
-F 1 "ATMEGA32-A" H 4625 1200 40  0000 L BNN
+F 1 "ATMEGA16" H 4625 1200 40  0000 L BNN
 F 2 "TQFP44" H 4175 3150 30  0000 C CIN
 F 3 "" H 4175 3150 60  0000 C CNN
